File: telemetria_receiver_2022/can.sch (KiCad schematic (older format))
At the start: 8 parts, among them U4 ATA6561-GAQW-N

Commit message: added logos lib, fixed routing, impedance matching of spi and sdio, removed external RTC, PCB rearrangement
Parts:
- FB2, FB3: symbol PUTM_KICAD_SYMBOLS:Ferrite_Bead_Small_PWR -> telemetria_receiver_2022-rescue:Ferrite_Bead_Small_PWR-PUTM_KICAD_SYMBOLS
Changed lines of the file:
@@
 EESchema Schematic File Version 4
-EELAYER 30 0
+LIBS:telemetria_receiver_2022-cache
+EELAYER 29 0
 EELAYER END
 $Descr A4 11693 8268
@@
 	4850 5150 5000 5150
 $Comp
-L PUTM_KICAD_SYMBOLS:Ferrite_Bead_Small_PWR FB?
+L telemetria_receiver_2022-rescue:Ferrite_Bead_Small_PWR-PUTM_KICAD_SYMBOLS FB?
 U 1 1 61BAD549
 P 2350 3850
@@
 $EndComp
 $Comp
-L PUTM_KICAD_SYMBOLS:Ferrite_Bead_Small_PWR FB?
+L telemetria_receiver_2022-rescue:Ferrite_Bead_Small_PWR-PUTM_KICAD_SYMBOLS FB?
 U 1 1 61BAD9FD
 P 4300 3850
